File: a.brd (EAGLE design)
At the start: 67.2 x 42.2 mm, 23 parts, among them SW1 TS6601-9,5, SW2 TS6601-9,5, U1 ESP32-WROVER-IE, X1 PLS-09, X2 PLS-07, X3 PLS2-6, X4 PLD-06

Commit message: more import
Parts:
- removed U1: ESP32-WROVER-IE, pds019_lit:ESP32-WROVER-E
- added MODULE1: ESP32-WROVER-(I)E, ali_modules:ESP32-WROVER-E
- C1: value 100,0 10V -> 100u; device pds019_lit:CTANT_TYPE_C -> rc:CTANT_TYPE_C
- C2, C3, C4: value 0,1 -> 0.1u; device pds019_lit:C0603 -> rc:C0603
- HL1, HL2: value FYLS-3528RGBC -> LED_RGB-3528; device pds019_lit:LED_3528_4P -> rc:LED3528
- R1, R2, R3, R4, R5, R6, R7, R8: device pds019_lit:R0603 -> rc:R0603
- RN1: device pds019_lit:RN_YC164 -> rc:R_4X0603
- SW1, SW2: device pds019_lit:SW4-6.0X6.0X5.0MM -> mechanical:SW4-6.0X6.0X5.0MM
- X1: value PLS-09 -> PINHEAD_1X09-2.54-TH-MALE; device pds019_lit:PLS-09 -> pinhead:1X09-PTH-2.54
- X2: value PLS-07 -> PINHEAD_1X07-2.54; device pds019_lit:PLS-07 -> pinhead:1X07-PTH-2.54
- X3: value PLS2-6 -> PINHEAD_1X06-2-MALE; device pds019_lit:PLS2-6 -> pinhead:1X06-PTH-2
- X4: value PLD-06 -> PINHEAD_2X03-PTH-2.54; device pds019:PLD-06 -> pinhead:2X03-PTH-2.54
- flipped X2 to the top
- turned RN1 to 90 degrees
- turned X4 to 90 degrees
Connections:
- removed net +3V3: C1.+, C2.2, HL1.2, HL2.2, R1.2, R2.2, U1.2, X1.2, X2.1, X3.2, X4.1
- new net VDD_3V3: C1.+, C2.2, HL1.2, HL2.2, MODULE1.2, R1.2, R2.2, X1.2, X2.1, X3.2, X4.1
- net !LED1_B: now also MODULE1.36; no longer U1.36
- net !LED1_G: now also MODULE1.33; no longer U1.33
- net !LED1_R: now also MODULE1.37; no longer U1.37
- net !LED2_B: now also MODULE1.30; no longer U1.30
- net !LED2_G: now also MODULE1.29; no longer U1.29
- net !LED2_R: now also MODULE1.31; no longer U1.31
- net ESP_BOOT: now also MODULE1.25; no longer U1.25
- net ESP_EN: now also MODULE1.3; no longer U1.3
- net ESP_IO2: now also MODULE1.24; no longer U1.24
- net ESP_IO35: now also MODULE1.7; no longer U1.7
- net ESP_IO39: now also MODULE1.5; no longer U1.5
- net ESP_IO4: now also MODULE1.26; no longer U1.26
- net ESP_RXD0: now also MODULE1.34; no longer U1.34
- net ESP_TXD0: now also MODULE1.35; no longer U1.35
- net EXT_SW: now also MODULE1.6; no longer U1.6
- net GND: now also MODULE1.1, MODULE1.15, MODULE1.38, MODULE1.39; no longer U1.1, U1.15, U1.38, U1.39
- net MTCK: now also MODULE1.16; no longer U1.16
- net MTDI: now also MODULE1.14; no longer U1.14
- net MTDO: now also MODULE1.23; no longer U1.23
- net MTMS: now also MODULE1.13; no longer U1.13
- net PWM_B: now also MODULE1.10; no longer U1.10
- net PWM_EN: now also MODULE1.12; no longer U1.12
- net PWM_G: now also MODULE1.9; no longer U1.9
- net PWM_R: now also MODULE1.8; no longer U1.8
- net PWM_W: now also MODULE1.11; no longer U1.11
- net SW_SETUP: now also MODULE1.4; no longer U1.4
Routing:
- net +3V3: track 152.1 -> 0.00 mm
- net VDD_3V3: track 0.00 -> 146.8 mm
- net MTDO: track 38.4 -> 34.7 mm
- net N$9: track 11.0 -> 8.40 mm
- net ESP_BOOT: track 23.8 -> 21.4 mm
- net PWM_EN: track 37.2 -> 35.0 mm
- net N$4: track 11.4 -> 9.33 mm
- net ESP_TXD0: track 34.1 -> 32.7 mm
- net MTCK: track 9.62 -> 8.27 mm
- net !LED1_G: track 49.7 -> 48.5 mm
- net MTDI: track 9.83 -> 8.83 mm
- net !LED2_R: track 48.8 -> 47.9 mm
- net ESP_RXD0: track 34.2 -> 33.3 mm
- net EXT_SW: track 34.5 -> 33.8 mm
- net !LED1_R: track 48.4 -> 47.6 mm
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Other:
- board text added: "PDS019_RGWB_A"
- board text removed: ">DRAWING_NAME"
- board text removed: ">PLOT_DATE_TIME"
